Commit message: mobile_manipulation2 works in gazeba

File: catkin_ws/src/piper_ros/src/mobile_manipulator2_description/piper_description/urdf/piper_description.urdf (robot description, URDF)
Before this commit: robot piper, 11 links, 10 joints
Links:
- removed link dummy_link
- added link dummy_root
- added link world
Joints:
- removed joint base_to_dummy
- added joint base_to_world: type fixed, parent dummy_root, child base_link, origin xyz=0 0 0 rpy=0 0 0
- added joint dummy_joint: type fixed, parent world, child dummy_root, origin xyz=0 0 0 rpy=0 0 0

File: catkin_ws/src/piper_ros/src/mobile_manipulator2_description/urdf/mobile_manipulator2_description.urdf (robot description, URDF)
Before this commit: robot mobile_manipulator2, 29 links, 27 joints
Links:
- added link dummy_root
- link arm_base_link: geometry collision mesh filename=package://mobile_manipulator2_description/piper_description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; visual mesh filename=package://mobile_manipulator2_description/piper_description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
- link arm_gripper_base: geometry collision mesh filename=package://mobile_manipulator2_description/piper_description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; visual mesh filename=package://mobile_manipulator2_description/piper_description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
- link arm_link1: geometry collision mesh filename=package://mobile_manipulator2_description/piper_description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; visual mesh filename=package://mobile_manipulator2_description/piper_description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
- link arm_link2: geometry collision mesh filename=package://mobile_manipulator2_description/piper_description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; visual mesh filename=package://mobile_manipulator2_description/piper_description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
- link arm_link3: geometry collision mesh filename=package://mobile_manipulator2_description/piper_description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; visual mesh filename=package://mobile_manipulator2_description/piper_description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
- link arm_link4: geometry collision mesh filename=package://mobile_manipulator2_description/piper_description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; visual mesh filename=package://mobile_manipulator2_description/piper_description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
- link arm_link5: geometry collision mesh filename=package://mobile_manipulator2_description/piper_description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; visual mesh filename=package://mobile_manipulator2_description/piper_description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
- link arm_link6: geometry collision mesh filename=package://mobile_manipulator2_description/piper_description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; visual mesh filename=package://mobile_manipulator2_description/piper_description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
- link arm_link7: geometry collision mesh filename=package://mobile_manipulator2_description/piper_description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; visual mesh filename=package://mobile_manipulator2_description/piper_description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
- link arm_link8: geometry collision mesh filename=package://mobile_manipulator2_description/piper_description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; visual mesh filename=package://mobile_manipulator2_description/piper_description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
- link base_link: geometry collision mesh filename=package://mobile_manipulator2_description/meshes/base_link.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; visual mesh filename=package://mobile_manipulator2_description/meshes/base_link.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
- link left_Link: geometry collision mesh filename=package://mobile_manipulator2_description/meshes/left_Link.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; visual mesh filename=package://mobile_manipulator2_description/meshes/left_Link.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
- link left_front_link: geometry collision mesh filename=package://mobile_manipulator2_description/meshes/left_front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; visual mesh filename=package://mobile_manipulator2_description/meshes/left_front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
- link left_rear_link: geometry collision mesh filename=package://mobile_manipulator2_description/meshes/left_rear_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; visual mesh filename=package://mobile_manipulator2_description/meshes/left_rear_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
- link right_front_link: geometry collision mesh filename=package://mobile_manipulator2_description/meshes/right_fron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; visual mesh filename=package://mobile_manipulator2_description/meshes/right_fron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
- link right_link: geometry collision mesh filename=package://mobile_manipulator2_description/meshes/right_link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; visual mesh filename=package://mobile_manipulator2_description/meshes/right_link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
- link right_rear_link: geometry collision mesh filename=package://mobile_manipulator2_description/meshes/right_rear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; visual mesh filename=package://mobile_manipulator2_description/meshes/right_rear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
Joints:
- added joint dummy_joint: type fixed, parent dummy_root, child base_link, origin xyz=0 0 0 rpy=0 0 0
- added joint front_camera_pole_to_mount: type fixed, parent FrontCamera_vertical_pole, child FrontCamera_mount, origin xyz=0 0 0.03 rpy=0 0 0

Commit message: v1.0: real urdf and moveit done

File: catkin_ws/src/piper_ros/src/mobile_manipulator2_description/piper_description/urdf/piper_description.urdf (robot description, URDF)
Before this commit: robot piper, 12 links, 11 joints
Links:
- removed link dummy_root
- removed link world
- added link dummy_link
Joints:
- removed joint base_to_world
- removed joint dummy_joint
- added joint base_to_dummy: type fixed, parent dummy_link, child base_link, origin xyz=0 0 0 rpy=0 0 0
- joint joint1: limit lower=-2.618 upper=2.618 effort=100 velocity=5 -> lower=-2.618 upper=2.168 effort=100 velocity=5
- joint joint7: limit lower=0 upper=0.035 effort=100 velocity=1 -> lower=0 upper=0.035 effort=10 velocity=1
- joint joint8: limit lower=-0.035 upper=0 effort=100 velocity=1 -> lower=-0.035 upper=0 effort=10 velocity=1

File: catkin_ws/src/piper_ros/src/mobile_manipulator2_description/piper_description/urdf/piper_description.xacro (robot description, xacro)
@@ -4,12 +4,12 @@
   xmlns:xacro="http://ros.org/wiki/xacro">
 <!-- world -->
-  <link name="world"/>
+  <!-- <link name="world"/>
   <joint name="fixed_base_joint" type="fixed">
       <parent link="world"/>
       <child link="base_link"/>
-  </joint>
+  </joint> -->
 <!-- piper -->
 <link
-    name="base_link">
+    name="arm_base">
     <inertial>
       <origin
@@ -97,5 +97,5 @@
       rpy="0 0 0" />
     <parent
-      link="base_link" />
+      link="arm_base" />
     <child
       link="link1" />
@@ -104,5 +104,5 @@
     <limit
       lower="-2.618"
-      upper="2.618"
+      upper="2.168"
       effort="100"
       velocity="5" />
@@ -506,5 +506,5 @@
       lower="0"
       upper="0.035"
-      effort="100"
+      effort="10"
       velocity="1" />
   </joint>
@@ -564,5 +564,5 @@
       lower="-0.035"
       upper="0"
-      effort="100"
+      effort="10"
       velocity="1" />
   </joint>

File: catkin_ws/src/piper_ros/src/mobile_manipulator2_description/piper_description/urdf/piper_description_gazebo.xacro (robot description, xacro)
@@ -104,5 +104,5 @@
     <limit
       lower="-2.618"
-      upper="2.618"
+      upper="2.168"
       effort="100"
       velocity="5" />

File: catkin_ws/src/piper_ros/src/mobile_manipulator2_description/piper_description/urdf/piper_description_old.urdf (robot description, URDF)
Before this commit: robot piper, 10 links, 9 joints
Joints:
- joint joint1: limit lower=-2.618 upper=2.618 effort=100 velocity=5 -> lower=-2.618 upper=2.168 effort=100 velocity=5
- joint joint7: limit lower=0 upper=0.035 effort=100 velocity=1 -> lower=0 upper=0.035 effort=10 velocity=1
- joint joint8: limit lower=-0.035 upper=0 effort=100 velocity=1 -> lower=-0.035 upper=0 effort=10 velocity=1

File: catkin_ws/src/piper_ros/src/mobile_manipulator2_description/piper_description/urdf/piper_no_gripper_description.urdf (robot description, URDF)
Before this commit: robot piper, 8 links, 7 joints
Joints:
- joint joint1: limit lower=-2.618 upper=2.618 effort=100 velocity=5 -> lower=-2.618 upper=2.168 effort=100 velocity=5

File: catkin_ws/src/piper_ros/src/mobile_manipulator2_description/piper_description/urdf/piper_no_gripper_description.xacro (robot description, xacro)
@@ -104,5 +104,5 @@
     <limit
       lower="-2.618"
-      upper="2.618"
+      upper="2.168"
       effort="100"
       velocity="5" />

File: catkin_ws/src/piper_ros/src/mobile_manipulator2_description/piper_description/urdf/piper_no_gripper_description_gazebo.xacro (robot description, xacro)
@@ -104,5 +104,5 @@
     <limit
       lower="-2.618"
-      upper="2.618"
+      upper="2.168"
       effort="100"
       velocity="5" />

File: catkin_ws/src/piper_ros/src/mobile_manipulator2_description/piper_description/urdf/piper_no_gripper_description_old.urdf (robot description, URDF)
Before this commit: robot piper, 7 links, 6 joints
Joints:
- joint joint1: limit lower=-2.618 upper=2.618 effort=100 velocity=5 -> lower=-2.618 upper=2.168 effort=100 velocity=5
