Commit message: feat: 根据实际硬件规格优化机械臂关节参数
更新机械臂关节运动范围和速度限制，使配置与实际硬件完全匹配:

关节运动范围更新:
- J1: ±154° (±2.687 rad)
- J2: 0°~195° (0~3.403 rad)
- J3: -175°~0° (-3.054~0 rad)
- J4: -102°~102° (-1.780~1.780 rad)
- J5: -75°~75° (-1.309~1.309 rad)
- J6: ±120° (±2.094 rad)

关节最大速度更新:
- J1: 180°/s (3.142 rad/s)
- J2: 195°/s (3.403 rad/s)
- J3: 180°/s (3.142 rad/s)
- J4-J6: 225°/s (3.927 rad/s)

更新的文件:
- URDF文件: piper_description.urdf, piper_no_gripper_description.urdf
- Xacro文件: piper_description.xacro, piper_no_gripper_description.xacro
- MoveIt配置: joint_limits.yaml (带夹爪和无夹爪版本)

新增工具:
- 验证脚本: _cc_verify_joint_limits.py
- 更新文档: joint_limits_update_summary.md

这些更新确保了机械臂在安全范围内运动，提升了运动规划的精确性。

🤖 Generated with [Claude Code](https://claude.ai/code)

Co-Authored-By: Claude <noreply@anthropic.com>

File: src/robot_description/piper_description/urdf/piper_description.urdf (robot description, URDF)
Before this commit: robot piper, 11 links, 10 joints
Joints:
- joint joint1: limit lower=-2.618 upper=2.168 effort=100 velocity=5 -> lower=-2.687 upper=2.687 effort=100 velocity=3.142
- joint joint2: limit lower=0 upper=3.14 effort=100 velocity=5 -> lower=0 upper=3.403 effort=100 velocity=3.403
- joint joint3: limit lower=-2.967 upper=0 effort=100 velocity=5 -> lower=-3.054 upper=0 effort=100 velocity=3.142
- joint joint4: limit lower=-1.745 upper=1.745 effort=100 velocity=5 -> lower=-1.780 upper=1.780 effort=100 velocity=3.927
- joint joint5: limit lower=-1.22 upper=1.22 effort=100 velocity=5 -> lower=-1.309 upper=1.309 effort=100 velocity=3.927
- joint joint6: limit lower=-2.0944 upper=2.0944 effort=100 velocity=3 -> lower=-2.094 upper=2.094 effort=100 velocity=3.927

File: src/robot_description/piper_description/urdf/piper_description.xacro (robot description, xacro)
@@ -103,8 +103,8 @@
       xyz="0 0 1" />
     <limit
-      lower="-2.618"
-      upper="2.168"
+      lower="-2.687"
+      upper="2.687"
       effort="100"
-      velocity="5" />
+      velocity="3.142" />
   </joint>
   <link
@@ -163,7 +163,7 @@
     <limit
       lower="0"
-      upper="3.14"
+      upper="3.403"
       effort="100"
-      velocity="5" />
+      velocity="3.403" />
   </joint>
   <link
@@ -221,8 +221,8 @@
       xyz="0 0 1" />
     <limit
-      lower="-2.967"
+      lower="-3.054"
       upper="0"
       effort="100"
-      velocity="5" />
+      velocity="3.142" />
   </joint>
   <link
@@ -279,8 +279,8 @@
       xyz="0 0 1" />
     <limit
-      lower="-1.745"
-      upper="1.745"
+      lower="-1.780"
+      upper="1.780"
       effort="100"
-      velocity="5" />
+      velocity="3.927" />
   </joint>
   <link
@@ -337,8 +337,8 @@
       xyz="0 0 1" />
     <limit
-      lower="-1.22"
-      upper="1.22"
+      lower="-1.309"
+      upper="1.309"
       effort="100"
-      velocity="5" />
+      velocity="3.927" />
   </joint>
   <link
@@ -395,8 +395,8 @@
       xyz="0 0 1" />
     <limit
-      lower="-2.0944"
-      upper="2.0944"
+      lower="-2.094"
+      upper="2.094"
       effort="100"
-      velocity="3" />
+      velocity="3.927" />
   </joint>
   <link

File: src/robot_description/piper_description/urdf/piper_no_gripper_description.urdf (robot description, URDF)
Before this commit: robot piper, 8 links, 7 joints
Joints:
- joint joint1: limit lower=-2.618 upper=2.168 effort=100 velocity=5 -> lower=-2.687 upper=2.687 effort=100 velocity=3.142
- joint joint2: limit lower=0 upper=3.14 effort=100 velocity=5 -> lower=0 upper=3.403 effort=100 velocity=3.403
- joint joint3: limit lower=-2.967 upper=0 effort=100 velocity=5 -> lower=-3.054 upper=0 effort=100 velocity=3.142
- joint joint4: limit lower=-1.745 upper=1.745 effort=100 velocity=5 -> lower=-1.780 upper=1.780 effort=100 velocity=3.927
- joint joint5: limit lower=-1.22 upper=1.22 effort=100 velocity=5 -> lower=-1.309 upper=1.309 effort=100 velocity=3.927
- joint joint6: limit lower=-2.0944 upper=2.0944 effort=100 velocity=3 -> lower=-2.094 upper=2.094 effort=100 velocity=3.927

File: src/robot_description/piper_description/urdf/piper_no_gripper_description.xacro (robot description, xacro)
@@ -103,8 +103,8 @@
       xyz="0 0 1" />
     <limit
-      lower="-2.618"
-      upper="2.168"
-      effort="100"
-      velocity="5" />
+      lower="-2.687"
+      upper="2.687"
+      effort="100"
+      velocity="3.142" />
   </joint>
   <link
@@ -163,7 +163,7 @@
     <limit
       lower="0"
-      upper="3.14"
-      effort="100"
-      velocity="5" />
+      upper="3.403"
+      effort="100"
+      velocity="3.403" />
   </joint>
   <link
@@ -221,8 +221,8 @@
       xyz="0 0 1" />
     <limit
-      lower="-2.967"
+      lower="-3.054"
       upper="0"
       effort="100"
-      velocity="5" />
+      velocity="3.142" />
   </joint>
   <link
@@ -279,8 +279,8 @@
       xyz="0 0 1" />
     <limit
-      lower="-1.745"
-      upper="1.745"
-      effort="100"
-      velocity="5" />
+      lower="-1.780"
+      upper="1.780"
+      effort="100"
+      velocity="3.927" />
   </joint>
   <link
@@ -337,8 +337,8 @@
       xyz="0 0 1" />
     <limit
-      lower="-1.22"
-      upper="1.22"
-      effort="100"
-      velocity="5" />
+      lower="-1.309"
+      upper="1.309"
+      effort="100"
+      velocity="3.927" />
   </joint>
   <link
@@ -395,8 +395,8 @@
       xyz="0 0 1" />
     <limit
-      lower="-2.0944"
-      upper="2.0944"
-      effort="100"
-      velocity="3" />
+      lower="-2.094"
+      upper="2.094"
+      effort="100"
+      velocity="3.927" />
   </joint>
 <!-- controller -->
