Commit message: fix: 调整under_camera位置到lidar顶部
- 将under_camera从base_link前方移动到lidar顶部
- parent link从base_link改为lidar_Link
- 新位置：lidar中心前方2.5cm，上方10cm
- 添加display_urdf.launch用于直接加载URDF文件

🤖 Generated with [Claude Code](https://claude.ai/code)

Co-Authored-By: Claude <noreply@anthropic.com>

File: src/robot_desc/mobile_manipulator2_description/urdf/mobile_manipulator2_description.urdf (robot description, URDF)
Before this commit: robot mobile_manipulator2, 16 links, 15 joints
Joints:
- joint under_camera_joint: origin xyz=0.35023 0 -0.00085446 rpy=0 0 0 -> xyz=0.025 0 0.1 rpy=0 0 0; parent base_link -> lidar_Link

Commit message: feat: Make mobile_manipulator2_description independent of piper_description
- Copy all piper mesh files to local directory with piper_ prefix
- Update URDF files to use local mesh copies instead of piper_description references
- Organize meshes into visual/ and collision/ subdirectories
- Keep link6 using camera_v3.dae as it represents the camera module

This eliminates the implicit dependency on piper_description package,
making mobile_manipulator2_description fully self-contained.

🤖 Generated with [Claude Code](https://claude.ai/code)

Co-Authored-By: Claude <noreply@anthropic.com>

File: src/robot_desc/mobile_manipulator2_description/urdf/mobile_manipulator2_description.urdf (robot description, URDF)
Before this commit: robot mobile_manipulator2, 16 links, 15 joints
Links:
- link arm_base: geometry collision mesh filename=package://mobile_manipulator2_description/meshes/visual/stl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; visual mesh filename=package://mobile_manipulator2_description/meshes/visual/dae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
- link link1: geometry collision mesh filename=package://mobile_manipulator2_description/meshes/visual/stl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; visual mesh filename=package://mobile_manipulator2_description/meshes/visual/dae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
- link link2: geometry collision mesh filename=package://mobile_manipulator2_description/meshes/visual/stl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; visual mesh filename=package://mobile_manipulator2_description/meshes/visual/dae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
- link link3: geometry collision mesh filename=package://mobile_manipulator2_description/meshes/visual/stl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; visual mesh filename=package://mobile_manipulator2_description/meshes/visual/dae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
- link link4: geometry collision mesh filename=package://mobile_manipulator2_description/meshes/visual/stl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; visual mesh filename=package://mobile_manipulator2_description/meshes/visual/dae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
- link link5: geometry collision mesh filename=package://mobile_manipulator2_description/meshes/visual/stl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; visual mesh filename=package://mobile_manipulator2_description/meshes/visual/dae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
- link link6: geometry collision mesh filename=package://mobile_manipulator2_description/meshes/visual/dae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; visual mesh filename=package://mobile_manipulator2_description/meshes/visual/dae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
- link link7: geometry collision mesh filename=package://mobile_manipulator2_description/meshes/visual/stl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; visual mesh filename=package://mobile_manipulator2_description/meshes/visual/dae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
- link link8: geometry collision mesh filename=package://mobile_manipulator2_description/meshes/visual/stl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; visual mesh filename=package://mobile_manipulator2_description/meshes/visual/dae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

Commit message: feat: Implement dual RGBD depth projection system with calibration and URDF methods
Major improvements:
- Added dual projection methods (calibration vs URDF-based)
- Implemented CameraDepthProjector with unified interface
- Added complete camera TF chain publishing system
- Created comprehensive testing framework
- Fixed camera intrinsics configuration (640x480 preferred)

Key features:
- src/perception/scripts/depth_projector_core.py: Core projection engine
- src/perception/launch/depth_projection.launch: Complete launch system
- src/robot_drivers/camera_driver/scripts/camera_tf_publisher.py: TF publisher
- Camera calibration configs with proper extrinsics
- Multi-camera support (hand, top, chassis)
- RViz visualization configs

Testing results:
- Calibration method: ✅ Working (fx=598.6, 640x480)
- URDF method: ✅ Architecture ready
- Unified interface eliminates special cases (Linus "good taste")

🤖 Generated with [Claude Code](https://claude.ai/code)

Co-Authored-By: Claude <noreply@anthropic.com>

File: src/robot_desc/mobile_manipulator2_description/urdf/mobile_manipulator2_description.urdf (robot description, URDF)
Before this commit: robot mobile_manipulator2, 16 links, 15 joints
Links:
- removed link box_Link
- removed link hand_cam
- removed link lidar_Link
- removed link lifting_Link
- removed link top_camera_Link
- removed link under_camera_Link
- added link box_link, mass 1.96086062558564; collision mesh filename=package://mobile_manipulator2_description/meshes/visual/box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; visual mesh filename=package://mobile_manipulator2_description/meshes/visual/box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
- added link chassis_camera_link, mass 0.055353; collision mesh filename=package://mobile_manipulator2_description/meshes/visual/top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; visual mesh filename=package://mobile_manipulator2_description/meshes/visual/top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
- added link hand_camera_link, mass 0.0067926; collision box size=0.02 0.08 0.02; visual box size=0.02 0.08 0.02
- added link lidar_link, mass 0.11388; collision mesh filename=package://mobile_manipulator2_description/meshes/visual/lid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; visual mesh filename=package://mobile_manipulator2_description/meshes/visual/lid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
- added link lifting_link, mass 1.28345031134681; collision mesh filename=package://mobile_manipulator2_description/meshes/visual/lif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; visual mesh filename=package://mobile_manipulator2_description/meshes/visual/lif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
- added link top_camera_link, mass 0.028999; collision mesh filename=package://mobile_manipulator2_description/meshes/visual/top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; visual mesh filename=package://mobile_manipulator2_description/meshes/visual/top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
- link base_link: geometry collision mesh filename=package://mobile_manipulator2_description/meshes/visual/cha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; visual mesh filename=package://mobile_manipulator2_description/meshes/visual/cha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
Joints:
- removed joint under_camera_joint
- added joint chassis_camera_joint: type fixed, parent lidar_link, child chassis_camera_link, origin xyz=0.025 0 0.1 rpy=0 0 0, axis 0 0 0
- joint arm_joint: parent box_Link -> box_link
- joint box_joint: child box_Link -> box_link
- joint hand_camera_joint: child hand_cam -> hand_camera_link; origin xyz=0.0 0.075 0.03 rpy=0 -0.3 1.57 -> xyz=0.0 0.075 0.03 rpy=0.000000 -0.7855105 -1.571021
- joint lidar_joint: child lidar_Link -> lidar_link
- joint lifting_joint: child lifting_Link -> lifting_link; parent box_Link -> box_link
- joint top_camera_joint: child top_camera_Link -> top_camera_link; parent lifting_Link -> lifting_link

File: src/robot_desc/mobile_manipulator2_description/urdf/mobile_manipulator2_performance.urdf (robot description, URDF)
Before this commit: robot mobile_manipulator2, 16 links, 15 joints
Links:
- removed link box_Link
- removed link hand_cam
- removed link lidar_Link
- removed link lifting_Link
- removed link top_camera_Link
- removed link under_camera_Link
- added link box_link, mass 1.96086062558564; collision mesh filename=package://mobile_manipulator2_description/meshes/collision/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; visual mesh filename=package://mobile_manipulator2_description/meshes/visual/box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
- added link chassis_camera_link, mass 0.055353; collision mesh filename=package://mobile_manipulator2_description/meshes/collision/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; visual mesh filename=package://mobile_manipulator2_description/meshes/visual/cha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
- added link hand_camera_link, mass 0.0067926; collision mesh filename=package://mobile_manipulator2_description/meshes/collision/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; visual box size=0.02 0.08 0.02
- added link lidar_link, mass 0.11388; collision mesh filename=package://mobile_manipulator2_description/meshes/collision/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; visual mesh filename=package://mobile_manipulator2_description/meshes/visual/lid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
- added link lifting_link, mass 1.28345031134681; collision mesh filename=package://mobile_manipulator2_description/meshes/collision/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; visual mesh filename=package://mobile_manipulator2_description/meshes/visual/lif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
- added link top_camera_link, mass 0.028999; collision mesh filename=package://mobile_manipulator2_description/meshes/collision/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; visual mesh filename=package://mobile_manipulator2_description/meshes/visual/top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
Joints:
- removed joint under_camera_joint
- added joint chassis_camera_joint: type fixed, parent lidar_link, child chassis_camera_link, origin xyz=0.025 0 0.1 rpy=0 0 0, axis 0 0 0
- joint arm_joint: parent box_Link -> box_link
- joint box_joint: child box_Link -> box_link
- joint hand_camera_joint: child hand_cam -> hand_camera_link; origin xyz=0.0 0.075 0.03 rpy=0 -0.3 1.57 -> xyz=0.0 0.075 0.03 rpy=0.000000  -0.7855105 -1.571021
- joint lidar_joint: child lidar_Link -> lidar_link
- joint lifting_joint: child lifting_Link -> lifting_link; parent box_Link -> box_link
- joint top_camera_joint: child top_camera_Link -> top_camera_link; parent lifting_Link -> lifting_link

File: src/robot_desc/piper_description/urdf/piper_description_v100_camera.urdf (robot description, URDF)
Before this commit: robot piper_camera, 10 links, 9 joints
Joints:
- joint hand_camera_joint: origin xyz=0.0 0.075 0.03 rpy=0 -0.3 1.57  -> xyz=0.0 0.075 0.03 rpy=0 1.27 1.57 
